File: MCU_STM32.kicad_sch (KiCad schematic)
At the start: 19 parts, among them J2 Conn_01x05, U3 STM32G474RETx, Y1 ECS-80-12-33-JGN-TR3

Commit message: Update rail descriptions in schematic to match actual rail names.
Signed-off-by: Vincent Cadicamo <vcadicamo@icloud.com>
Other:
- title: (none) -> MCU_STM32
Changed lines of the file:
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@@
 	(generator_version "10.0")
 	(paper "A4")
+	(title_block
+		(title "MCU_STM32")
+		(date "2026-07-08")
+		(rev "1")
+	)
 	(text "RKM notation is used in this Schematic\nFor Example:\n4.7uF is 4u7\n100nF is 100n\n\nCapacitors (C11 through C17) are decoupling\nfor VDD, where C11 is for bulk decoupling\nand C12 through C17 is for each VDD and VBAT\n"
 		(exclude_from_sim no)
@@
 			)
 		)
-		(property "Description" "Power symbol creates a global label with name \"+3.3V\""
+		(property "Description" "Power symbol creates a global label with name \"NRST\""
 			(at 203.2 99.06 0)
 			(hide yes)
@@
 			)
 		)
-		(property "Description" "Power symbol creates a global label with name \"+3.3V\""
+		(property "Description" "Power symbol creates a global label with name \"+3.3VA\""
 			(at 78.74 29.21 0)
 			(hide yes)
@@
 			)
 		)
-		(property "Description" "Power symbol creates a global label with name \"+3.3V\""
+		(property "Description" "Power symbol creates a global label with name \"+3.3VA\""
 			(at 151.13 40.64 0)
 			(hide yes)
@@
 			)
 		)
-		(property "Description" "Power symbol creates a global label with name \"+3.3V\""
+		(property "Description" "Power symbol creates a global label with name \"+3.3VA\""
 			(at 106.68 59.69 0)
 			(hide yes)
@@
 			)
 		)
-		(property "Description" "Power symbol creates a global label with name \"+3.3V\""
+		(property "Description" "Power symbol creates a global label with name \"NRST\""
 			(at 111.76 64.77 0)
 			(hide yes)
