File: MCU_STM32.kicad_sch (KiCad schematic)
At the start: 19 parts, among them J2 Conn_01x05, U3 STM32G474RETx, Y1 ECS-80-12-33-JGN-TR3

Commit message: Added filter, transient and ESD based on application diagram. Changed global labels to rails.
Signed-off-by: Emily <124216516+epariag@users.noreply.github.com>
Connections:
- net FAULT: now reaches U3.10 (PC2)
- net ENABLE: now reaches U3.8 (PC0)
- net STANDBY: now reaches U3.9 (PC1)
