File: MCU_STM32.kicad_sch (KiCad schematic)
At the start: 19 parts, among them J2 Conn_01x05, U3 STM32G474RETx, Y1 ECS-80-12-33-JGN-TR3

Commit message: Wired the AS5047P Encoder to the STM32 for reading the Stepper position
Signed-off-by: Vincent Cadicamo <vcadicamo@icloud.com>
Connections:
- net PC9: now reaches U3.41 (PC9)
- net SPI3_SCK: now reaches U3.52 (PC10)
- net SPI3_MISO: now reaches U3.53 (PC11)
- net SPI3_MOSI: now reaches U3.54 (PC12)
