File: Stepper_ESC.kicad_sch (KiCad schematic)
At the start: 0 parts

Commit message: Wired the AS5047P Encoder to the STM32 for reading the Stepper position
Signed-off-by: Vincent Cadicamo <vcadicamo@icloud.com>
Other:
- sheet Encoder_Interface renamed AS5047P
Changed lines of the file:
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@@
 			(color 0 0 0 0)
 		)
-		(property "Sheetname" "Encoder_Interface"
+		(property "Sheetname" "AS5047P"
 			(at 91.44 71.6784 0)
 			(show_name yes)

Commit message: Added Hierarchical Labels connecting the SPI bus from the STM32 to the AS5047P
Signed-off-by: Vincent Cadicamo <vcadicamo@icloud.com>
Other:
- added sheet TMC5160_Driver1 (TMC5160_Driver.kicad_sch)
- sheet MCU_STM32 ports: added PC9, SPI3_MISO, SPI3_MOSI, SPI3_SCK; removed none
Changed lines of the file:
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@@
 	)
 	(sheet
-		(at 91.44 49.53)
+		(at 91.44 39.37)
 		(size 12.7 3.81)
 		(exclude_from_sim no)
@@
 		)
 		(property "Sheetname" "TMC5160_Driver"
-			(at 91.44 48.8184 0)
+			(at 91.44 38.6584 0)
 			(show_name yes)
 			(do_not_autoplace no)
@@
 		)
 		(property "Sheetfile" "TMC5160_Driver.kicad_sch"
-			(at 91.44 53.9246 0)
+			(at 91.44 43.7646 0)
 			(show_name no)
 			(do_not_autoplace no)
@@
 	)
 	(sheet
-		(at 91.44 38.1)
+		(at 125.73 48.26)
 		(size 12.7 3.81)
 		(exclude_from_sim no)
@@
 			(color 0 0 0 0)
 		)
+		(property "Sheetname" "TMC5160_Driver1"
+			(at 125.73 47.5484 0)
+			(show_name yes)
+			(do_not_autoplace no)
+			(effects
+				(font
+					(size 1.27 1.27)
+				)
+				(justify left bottom)
+			)
+		)
+		(property "Sheetfile" "TMC5160_Driver.kicad_sch"
+			(at 125.73 52.6546 0)
+			(show_name no)
+			(do_not_autoplace no)
+			(effects
+				(font
+					(size 1.27 1.27)
+				)
+				(justify left top)
+			)
+		)
+		(instances
+			(project "Stepper_ESC"
+				(path "/9271e9dc-3850-4149-b59f-a263c29a5edc"
+					(page "7")
+				)
+			)
+		)
+	)
+	(sheet
+		(at 21.59 31.75)
+		(size 34.29 30.48)
+		(exclude_from_sim no)
+		(in_bom yes)
+		(on_board yes)
+		(dnp no)
+		(fields_autoplaced yes)
+		(stroke
+			(width 0.1524)
+			(type solid)
+		)
+		(fill
+			(color 0 0 0 0)
+		)
 		(property "Sheetname" "MCU_STM32"
-			(at 91.44 37.3884 0)
+			(at 21.59 31.0384 0)
 			(show_name yes)
 			(do_not_autoplace no)
@@
 		)
 		(property "Sheetfile" "MCU_STM32.kicad_sch"
-			(at 91.44 42.4946 0)
-			(show_name no)
-			(do_not_autoplace no)
-			(effects
-				(font
-					(size 1.27 1.27)
-				)
-				(justify left top)
-			)
-		)
+			(at 21.59 62.8146 0)
+			(show_name no)
+			(do_not_autoplace no)
+			(effects
+				(font
+					(size 1.27 1.27)
+				)
+				(justify left top)
+			)
+		)
+		(pin "PC9" bidirectional
+			(at 55.88 33.02 0)
+			(effects
+				(font
+					(size 1.27 1.27)
+				)
+				(justify right)
+			)
+		)
+		(pin "SPI3_MISO" bidirectional
+			(at 55.88 43.18 0)
+			(effects
+				(font
+					(size 1.27 1.27)
+				)
+				(justify right)
+			)
+		)
+		(pin "SPI3_MOSI" bidirectional
+			(at 55.88 40.64 0)
+			(effects
+				(font
+					(size 1.27 1.27)
+				)
+				(justify right)
+			)
+		)
+		(pin "SPI3_SCK" bidirectional
+			(at 55.88 38.1 0)
+			(effects
+				(font
+					(size 1.27 1.27)
+				)
+				(justify right)
+			)
+		)
