File: Stepper_ESC.kicad_sch (KiCad schematic)
At the start: 0 parts

Commit message: Updated traces on PCB for the power supply, added XT60PW power connector for the board.
Other:
- removed sheet TMC5160_Driver5
Changed lines of the file:
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@@
-	)
-	(sheet
-		(at 82.55 143.51)
-		(size 29.21 12.7)
-		(exclude_from_sim no)
-		(in_bom yes)
-		(on_board yes)
-		(dnp no)
-		(fields_autoplaced yes)
-		(stroke
-			(width 0.1524)
-			(type solid)
-		)
-		(fill
-			(color 0 0 0 0)
-		)
-		(property "Sheetname" "TMC5160_Driver5"
-			(at 82.55 142.7984 0)
-			(show_name yes)
-			(do_not_autoplace no)
-			(effects
-				(font
-					(size 1.27 1.27)
-				)
-				(justify left bottom)
-			)
-		)
-		(property "Sheetfile" "TMC5160_Driver.kicad_sch"
-			(at 82.55 156.7946 0)
-			(show_name no)
-			(do_not_autoplace no)
-			(effects
-				(font
-					(size 1.27 1.27)
-				)
-				(justify left top)
-			)
-		)
-		(pin "CSN_CFG3" input
-			(at 82.55 146.05 180)
-			(effects
-				(font
-					(size 1.27 1.27)
-				)
-				(justify left)
-			)
-		)
-		(pin "SCK_CFG2" input
-			(at 82.55 148.59 180)
-			(effects
-				(font
-					(size 1.27 1.27)
-				)
-				(justify left)
-			)
-		)
-		(pin "SDI_CFG1" input
-			(at 82.55 151.13 180)
-			(effects
-				(font
-					(size 1.27 1.27)
-				)
-				(justify left)
-			)
-		)
-		(pin "SDO_CFG0" input
-			(at 82.55 153.67 180)
-			(effects
-				(font
-					(size 1.27 1.27)
-				)
-				(justify left)
-			)
-		)
-		(instances
-			(project "Stepper_ESC"
-				(path "/9271e9dc-3850-4149-b59f-a263c29a5edc"
-					(page "4")
-				)
-			)
-		)
 	)
 	(sheet
