File: TMC5160_Driver.kicad_sch (KiCad schematic)
At the start: 36 parts, among them J9 BLR-514-5-V, Q21 MCM3400A-TP, Q22 MCM3400A-TP, Q23 MCM3400A-TP, Q24 MCM3400A-TP, U11 TMC5160A-TA-T

Commit message: Updated traces on PCB for the power supply, added XT60PW power connector for the board.
Parts:
- renumbered C115 to C48, C114 to C49, C116 to C50, C121 to C51, C108 to C52, C113 to C53, C117 to C54, C120 to C55, C122 to C56, C109 to C57, C112 to C58, C110 to C59, C118 to C60, C119 to C61, C111 to C62, J9 to J5, Q21 to Q5, Q22 to Q6, Q23 to Q7, Q24 to Q8, R87 to R26, R90 to R27, R94 to R28, R97 to R29, R92 to R30, R99 to R31, R91 to R32, R93 to R33, R98 to R34, R100 to R35, R88 to R36, R89 to R37, R95 to R38, R96 to R39, R86 to R40, U11 to U7
