File: _restore_backup_2026-07-19T11-47-17-945/CAN_Interface.kicad_sch (KiCad schematic)
At the start: 15 parts, among them J4 Screw_Terminal_01x02, U5 TCAN1473-Q1

Commit message: Updated Footprints for PCB. Started footprint layout and trace routing
Signed-off-by: Vincent Cadicamo <vcadicamo@icloud.com>
Parts:
- D3, D4: footprint Diode_SMD:D_01005_0402Metric -> (none)
- J4: footprint TerminalBlock_MetzConnect:TerminalBlock_MetzConnect_Type011_RT05502HBLC_1x02_P5.00mm_Horizontal -> (none)
- R22, R23: footprint Resistor_SMD:R_01005_0402Metric -> (none)
- U5: footprint Stepper_ESC:D0014A-IPC_A -> footprints:D0014A-IPC_B
Changed lines of the file:
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@@
 			)
 		)
-		(property "Footprint" "Resistor_SMD:R_01005_0402Metric"
+		(property "Footprint" ""
 			(at 191.262 86.36 90)
 			(hide yes)
@@
 			)
 		)
-		(property "Footprint" "Resistor_SMD:R_01005_0402Metric"
+		(property "Footprint" ""
 			(at 191.262 97.79 90)
 			(hide yes)
@@
 			)
 		)
-		(property "Footprint" "TerminalBlock_MetzConnect:TerminalBlock_MetzConnect_Type011_RT05502HBLC_1x02_P5.00mm_Horizontal"
+		(property "Footprint" ""
 			(at 248.92 91.44 0)
 			(hide yes)
@@
 			)
 		)
-		(property "Footprint" "Diode_SMD:D_01005_0402Metric"
+		(property "Footprint" ""
 			(at 214.63 100.33 0)
 			(hide yes)
@@
 			)
 		)
-		(property "Footprint" "Stepper_ESC:D0014A-IPC_A"
+		(property "Footprint" "footprints:D0014A-IPC_B"
 			(at 149.86 90.17 0)
 			(hide yes)
@@
 			)
 		)
-		(property "Footprint" "Diode_SMD:D_01005_0402Metric"
+		(property "Footprint" ""
 			(at 214.63 83.82 0)
 			(hide yes)
