File: _restore_backup_2026-07-19T11-47-17-945/Encoder_Interface.kicad_sch (KiCad schematic)
At the start: 2 parts, among them U6 AS5047P-ATSM

Commit message: Updated Footprints for PCB. Started footprint layout and trace routing
Signed-off-by: Vincent Cadicamo <vcadicamo@icloud.com>
Parts:
- U6: footprint Stepper_ESC:TSSOP14_OSM -> TSSOP14_OSM
Changed lines of the file:
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@@
 			)
 		)
-		(property "Footprint" "Stepper_ESC:TSSOP14_OSM"
+		(property "Footprint" "TSSOP14_OSM"
 			(at 133.096 76.708 0)
 			(hide yes)
