File: _restore_backup_2026-07-19T11-47-17-945/MCU_STM32.kicad_sch (KiCad schematic)
At the start: 19 parts, among them J2 Conn_01x05, U3 STM32G474RETx, Y1 ECS-80-12-33-JGN-TR3

Commit message: Updated Footprints for PCB. Started footprint layout and trace routing
Signed-off-by: Vincent Cadicamo <vcadicamo@icloud.com>
Parts:
- FB1: footprint Inductor_SMD:L_01005_0402Metric -> (none)
Changed lines of the file:
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@@
 			)
 		)
-		(property "Footprint" "Inductor_SMD:L_01005_0402Metric"
+		(property "Footprint" ""
 			(at 76.962 24.13 90)
 			(hide yes)
