File: _restore_backup_2026-07-19T11-47-17-945/Power_Supply.kicad_sch (KiCad schematic)
At the start: 22 parts, among them J1 12V_Input, U1 TPS54360DDA, U2 AMS1117-3.3

Commit message: Updated Footprints for PCB. Started footprint layout and trace routing
Signed-off-by: Vincent Cadicamo <vcadicamo@icloud.com>
Parts:
- C9: footprint Capacitor_SMD:C_0402_1005Metric -> (none)
- D2: footprint Diode_SMD:D_01005_0402Metric -> (none)
- F1: footprint Fuse:Fuse_0402_1005Metric -> (none)
- J1: footprint Connector_PinSocket_2.00mm:PinSocket_1x02_P2.00mm_Horizontal -> (none)
Changed lines of the file:
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@@
 			)
 		)
-		(property "Footprint" "Capacitor_SMD:C_0402_1005Metric"
+		(property "Footprint" ""
 			(at 139.3952 82.55 0)
 			(hide yes)
@@
 			)
 		)
-		(property "Footprint" "Diode_SMD:D_01005_0402Metric"
+		(property "Footprint" ""
 			(at 60.96 27.94 0)
 			(hide yes)
@@
 			)
 		)
-		(property "Footprint" "Connector_PinSocket_2.00mm:PinSocket_1x02_P2.00mm_Horizontal"
+		(property "Footprint" ""
 			(at 62.23 55.88 0)
 			(hide yes)
@@
 			)
 		)
-		(property "Footprint" "Fuse:Fuse_0402_1005Metric"
+		(property "Footprint" ""
 			(at 78.74 54.102 90)
 			(hide yes)
